File: attiny_switch/attiny_switch.kicad_sch (KiCad schematic)
At the start: 11 parts, among them J1 12V in, J2 12V out, J3 UPDI Connector, J4 RPI_signal, U1 ATtiny1614-SS, U2 ISP772T

Commit message: PCB rev1
Parts:
- added C2: 100nF, Capacitor_SMD:C_1206_3216Metric, symbol Device:C
- added C3: 10uF, Capacitor_SMD:C_1206_3216Metric, symbol Device:C
- added D1: LED, LED_SMD:LED_1206_3216Metric, symbol Device:LED
- added H1, H2, H3: MountingHole, MountingHole:MountingHole_3.2mm_M3, symbol Mechanical:MountingHole
- added J5: Serial Connector, Connector_PinHeader_2.54mm:PinHeader_1x04_P2.54mm_Vertical, symbol Connector:Conn_01x04_Socket
- added J6: RPI Signal, TerminalBlock:TerminalBlock_MaiXu_MX126-5.0-02P_1x02_P5.00mm, symbol Connector:Conn_01x02_Socket
- added R5: 7,5k, Resistor_SMD:R_1206_3216Metric, symbol Device:R
- added SW1: SW_DPDT_x2, Connector_PinHeader_2.54mm:PinHeader_1x03_P2.54mm_Vertical, symbol Switch:SW_DPDT_x2
- added U3: Optocoupler, Package_DIP:DIP-4_W7.62mm, symbol Isolator:Optocoupler_DC_PhotoNPN_AKEC
- BT1: footprint (none) -> Eagle-12BH212P-GR:Untitled
- C1: footprint (none) -> Capacitor_SMD:C_1206_3216Metric
- J1, J2: footprint (none) -> TerminalBlock:TerminalBlock_MaiXu_MX126-5.0-02P_1x02_P5.00mm
- J3: footprint (none) -> Connector_PinHeader_2.54mm:PinHeader_1x03_P2.54mm_Vertical
- J4: value RPI_signal -> RPI Signal (OK); footprint (none) -> TerminalBlock:TerminalBlock_MaiXu_MX126-5.0-02P_1x02_P5.00mm
- R1, R3: footprint (none) -> Resistor_SMD:R_1206_3216Metric
- R2: value 1k -> 1k87; footprint (none) -> Resistor_SMD:R_1206_3216Metric
Connections:
- net at BT1.1 (+), J3.1 (Pin_1), R1.1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: now also C2.2, C3.1, J5.1 (Pin_1), SW1.1 (A)
- net GND: now reaches BT1.2 (-), C1.2, J1.2 (Pin_2), J2.2 (Pin_2), J3.3 (Pin_3), R3.1, U1.14 (GND), U2.1 (GND)
- net GND: now also C2.1, C3.2, D1.1 (K), J5.4 (Pin_4), J6.2 (Pin_2), U3.3; no longer J4.2 (Pin_2)
- net at R3.2, U1.11 (PA1): now also SW1.3 (C); no longer R2.2
- net at U1.12 (PA2): now also J6.1 (Pin_1), U3.4; no longer J4.1 (Pin_1)
- net at U1.6 (PB3): now also J5.3 (Pin_3)
- net at U1.7 (PB2): now also J5.2 (Pin_2)
- net at R2.1: now also J4.1 (Pin_1); no longer U2.2 (IN)
- net at J2.1 (Pin_1), U2.3 (OUT): now also R5.1
- new net: R2.2, U3.1
- new net: J4.2 (Pin_2), U3.2
- new net: D1.2 (A), R5.2
- new net: SW1.2 (B), U2.2 (IN)
Other:
- moved on the sheet: BT1, J1, J2, J3, J4, R1, R3, U1
